File: hardware/ascii_terminal_kicad.kicad_pcb (KiCad board)
At the start: 2 copper layers, 50.8 x 94 mm, 85 parts, among them J1 BOOT0, J2 5V, J3 VGA, J4 USB_KEYBOARD, J5 USB_COMM, J6 USB_POWER, J7 SERIAL, J8 SWDEBUG, SW1 RESET, U1 STM32F469VGTx, U2 LT1761-3.3, Y1 8MHz

Commit message: Cleanup tracks and vias
Connections:
- R10 pad 2: LTDC_R3 -> LTDC_R6
- R11 pad 2: LTDC_R4 -> LTDC_R5
- R12 pad 2: LTDC_R5 -> LTDC_R4
- R13 pad 2: LTDC_R6 -> LTDC_R3
- R14 pad 2: LTDC_R7 -> LTDC_R2
- R22 pad 2: LTDC_G2 -> LTDC_G7
- R23 pad 2: LTDC_G3 -> LTDC_G6
- R24 pad 2: LTDC_G4 -> LTDC_G5
- R25 pad 2: LTDC_G5 -> LTDC_G4
- R26 pad 2: LTDC_G6 -> LTDC_G3
- R27 pad 2: LTDC_G7 -> LTDC_G2
- R34 pad 2: LTDC_B2 -> LTDC_B7
- R35 pad 2: LTDC_B3 -> LTDC_B6
- R36 pad 2: LTDC_B4 -> LTDC_B5
- R37 pad 2: LTDC_B5 -> LTDC_B4
- R38 pad 2: LTDC_B6 -> LTDC_B3
- R39 pad 2: LTDC_B7 -> LTDC_B2
- R9 pad 2: LTDC_R2 -> LTDC_R7
Routing:
- net VDD: track 227.7 -> 0.00 mm
- net GND: track 174.9 -> 0.00 mm, vias 29 -> 0
- net +5VD: track 159.0 -> 0.00 mm
- net NRST: track 97.0 -> 0.00 mm, vias 2 -> 0
- net TRACESWO: track 67.0 -> 0.00 mm, vias 4 -> 0
- net LTDC_G2: track 63.2 -> 0.00 mm, vias 2 -> 0
- net LTDC_HSYNC: track 58.7 -> 0.00 mm, vias 2 -> 0
- net LTDC_R2: track 58.4 -> 0.00 mm, vias 2 -> 0
- net LTDC_B3: track 54.1 -> 0.00 mm, vias 2 -> 0
- net LTDC_R3: track 53.5 -> 0.00 mm, vias 2 -> 0
- net USB_OTG_FS_DM: track 52.2 -> 0.00 mm, vias 2 -> 0
- net LTDC_G3: track 51.5 -> 0.00 mm, vias 2 -> 0
- net LTDC_B2: track 50.5 -> 0.00 mm, vias 2 -> 0
- net USB_OTG_FS_DP: track 50.0 -> 0.00 mm, vias 2 -> 0
- net LTDC_B4: track 49.6 -> 0.00 mm, vias 2 -> 0
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
Commit message: Re-route
Routing:
- net VDD: track 0.00 -> 214.7 mm, vias 0 -> 7
- net GND: track 0.00 -> 185.5 mm, vias 0 -> 28
- net +5VD: track 0.00 -> 120.9 mm, vias 0 -> 2
- net NRST: track 0.00 -> 92.7 mm, vias 0 -> 4
- net LTDC_R7: track 0.00 -> 69.7 mm, vias 0 -> 2
- net LTDC_HSYNC: track 0.00 -> 67.6 mm, vias 0 -> 2
- net LTDC_R6: track 0.00 -> 64.6 mm, vias 0 -> 2
- net LTDC_B5: track 0.00 -> 61.4 mm, vias 0 -> 2
- net LTDC_B7: track 0.00 -> 58.8 mm, vias 0 -> 2
- net LTDC_R4: track 0.00 -> 54.8 mm, vias 0 -> 2
- net LTDC_G6: track 0.00 -> 53.5 mm, vias 0 -> 2
- net USB_OTG_FS_DM: track 0.00 -> 53.2 mm, vias 0 -> 2
- net LTDC_VSYNC: track 0.00 -> 51.6 mm, vias 0 -> 2
- net LTDC_G5: track 0.00 -> 51.3 mm, vias 0 -> 2
- net LTDC_B6: track 0.00 -> 51.1 mm, vias 0 -> 2
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Other:
- board text added: "Color Terminal 3.1 Copyright (C) 2019-2020 Peter Hizalev https://github.com/petrohi/ascii_terminal"
- board text removed: "Color ASCII Terminal 3.0 Copyright (C) 2019-2020 Peter Hizalev https://github.com/petrohi/ascii_terminal"
